Commit message: now editing urdf

File: robot.urdf (robot description, URDF)
Before this commit: robot go1, 37 links, 36 joints
Links:
- link FL_calf: geometry collision box size=0.213 0.016 0.016; visual mesh filename=package://go1_description/meshes/calf.dae scale=1 1 1
- link FL_hip: geometry collision cylinder length=0.04 radius=0.046; visual mesh filename=package://go1_description/meshes/hip.dae scale=1 1 1
- link FL_thigh: geometry collision box size=0.213 0.0245 0.034; visual mesh filename=package://go1_description/meshes/thigh.dae scale=1 1 1
- link FR_calf: geometry collision box size=0.213 0.016 0.016; visual mesh filename=package://go1_description/meshes/calf.dae scale=1 1 1
- link FR_hip: geometry collision cylinder length=0.04 radius=0.046; visual mesh filename=package://go1_description/meshes/hip.dae scale=1 1 1
- link FR_thigh: geometry collision box size=0.213 0.0245 0.034; visual mesh filename=package://go1_description/meshes/thigh_mirror.dae scale=1 1 1
- link RL_calf: geometry collision box size=0.213 0.016 0.016; visual mesh filename=package://go1_description/meshes/calf.dae scale=1 1 1
- link RL_hip: geometry collision cylinder length=0.04 radius=0.046; visual mesh filename=package://go1_description/meshes/hip.dae scale=1 1 1
- link RL_thigh: geometry collision box size=0.213 0.0245 0.034; visual mesh filename=package://go1_description/meshes/thigh.dae scale=1 1 1
- link RR_calf: geometry collision box size=0.213 0.016 0.016; visual mesh filename=package://go1_description/meshes/calf.dae scale=1 1 1
- link RR_hip: geometry collision cylinder length=0.04 radius=0.046; visual mesh filename=package://go1_description/meshes/hip.dae scale=1 1 1
- link RR_thigh: geometry collision box size=0.213 0.0245 0.034; visual mesh filename=package://go1_description/meshes/thigh_mirror.dae scale=1 1 1
- link optitrack_link: mass 1e-06 -> 1E-06
- link trunk_original: geometry collision box size=0.3 0.3 0.2; visual mesh filename=package://go1_description/meshes/skymul_go1_v2/base_link.STL
Joints:
- joint FL_calf_joint: axis 0.0 1.0 0.0 -> 0 1 0; origin xyz=0.0 0.0 -0.213 rpy=0.0 0.0 0.0 -> xyz=0 0 -0.213 rpy=0 0 0
- joint FL_foot_fixed: origin xyz=0.0 0.0 -0.213 rpy=0.0 0.0 0.0 -> xyz=0 0 -0.213 rpy=0 0 0
- joint FL_hip_joint: axis 1.0 0.0 0.0 -> 1 0 0; origin xyz=0.2118 0.13 0.0 rpy=0.0 0.0 0.0 -> xyz=0.2118 0.130 0 rpy=0 0 0
- joint FL_hip_rotor_joint: axis 0.0 0.0 0.0 -> 0 0 0; origin xyz=0.13 -0.145499999999996 0.0 rpy=-1.5707963267949 0.0 0.0 -> xyz=0.13 -0.145499999999996 0 rpy=-1.5707963267949 0 0
- joint FL_thigh_joint: axis 0.0 1.0 0.0 -> 0 1 0; origin xyz=0.0 0.08 0.0 rpy=0.0 0.0 0.0 -> xyz=0 0.08 0 rpy=0 0 0
- joint FR_calf_joint: axis 0.0 1.0 0.0 -> 0 1 0; origin xyz=0.0 0.0 -0.213 rpy=0.0 0.0 0.0 -> xyz=0 0 -0.213 rpy=0 0 0
- joint FR_foot_fixed: origin xyz=0.0 0.0 -0.213 rpy=0.0 0.0 0.0 -> xyz=0 0 -0.213 rpy=0 0 0
- joint FR_hip_joint: axis 1.0 0.0 0.0 -> 1 0 0; origin xyz=0.2118 -0.13 0.0 rpy=0.0 0.0 0.0 -> xyz=0.2118 -0.130 0 rpy=0 0 0
- joint FR_hip_rotor_joint: axis 0.0 0.0 0.0 -> 0 0 0; origin xyz=-0.13 -0.145499999999996 0.0 rpy=1.5707963267949 0.0 3.14159265358979 -> xyz=-0.13 -0.145499999999996 0 rpy=1.5707963267949 0 3.14159265358979
- joint FR_thigh_joint: axis 0.0 1.0 0.0 -> 0 1 0; origin xyz=0.0 -0.08 0.0 rpy=0.0 0.0 0.0 -> xyz=0 -0.08 0 rpy=0 0 0
- joint RL_calf_joint: axis 0.0 1.0 0.0 -> 0 1 0; origin xyz=0.0 0.0 -0.213 rpy=0.0 0.0 0.0 -> xyz=0 0 -0.213 rpy=0 0 0
- joint RL_foot_fixed: origin xyz=0.0 0.0 -0.213 rpy=0.0 0.0 0.0 -> xyz=0 0 -0.213 rpy=0 0 0
- joint RL_hip_joint: axis 1.0 0.0 0.0 -> 1 0 0; origin xyz=-0.2118 0.13 0.0 rpy=0.0 0.0 0.0 -> xyz=-0.2118 0.130 0 rpy=0 0 0
- joint RL_hip_rotor_joint: axis 0.0 0.0 0.0 -> 0 0 0; origin xyz=0.13 0.145500000000004 0.0 rpy=-1.5707963267949 0.0 3.14159265358979 -> xyz=0.13 0.145500000000004 0 rpy=-1.5707963267949 0 3.14159265358979
- joint RL_thigh_joint: axis 0.0 1.0 0.0 -> 0 1 0; origin xyz=0.0 0.08 0.0 rpy=0.0 0.0 0.0 -> xyz=0 0.08 0 rpy=0 0 0
- joint RR_calf_joint: axis 0.0 1.0 0.0 -> 0 1 0; origin xyz=0.0 0.0 -0.213 rpy=0.0 0.0 0.0 -> xyz=0 0 -0.213 rpy=0 0 0
- joint RR_foot_fixed: origin xyz=0.0 0.0 -0.213 rpy=0.0 0.0 0.0 -> xyz=0 0 -0.213 rpy=0 0 0
- joint RR_hip_joint: axis 1.0 0.0 0.0 -> 1 0 0; origin xyz=-0.2118 -0.13 0.0 rpy=0.0 0.0 0.0 -> xyz=-0.2118 -0.130 0 rpy=0 0 0
- joint RR_hip_rotor_joint: axis 0.0 0.0 0.0 -> 0 0 0; origin xyz=-0.13 0.1455 0.0 rpy=-1.5707963267949 0.0 3.14159265358979 -> xyz=-0.13 0.1455 0 rpy=-1.5707963267949 0 3.14159265358979
- joint RR_thigh_joint: axis 0.0 1.0 0.0 -> 0 1 0; origin xyz=0.0 -0.08 0.0 rpy=0.0 0.0 0.0 -> xyz=0 -0.08 0 rpy=0 0 0
- joint battery: axis 0.0 0.0 0.0 -> 0 0 0; origin xyz=-0.0375 0.18558 0.0938526402504663 rpy=0.0 1.5707963267949 0.0 -> xyz=-0.0375 0.18558 0.0938526402504663 rpy=0 1.5707963267949 0
- joint camera_color_joint: origin xyz=0.0 0.015 0.0 rpy=0.0 0.0 0.0 -> xyz=0 0.015 0 rpy=0 0 0
- joint camera_color_optical_joint: origin xyz=0.0 0.0 0.0 rpy=-1.5707963267948966 0.0 -1.5707963267948966 -> xyz=0 0 0 rpy=-1.5707963267948966 0 -1.5707963267948966
- joint camera_depth_joint: origin xyz=0.0 0.0 0.0 rpy=0.0 0.0 0.0 -> xyz=0 0 0 rpy=0 0 0
- joint camera_depth_optical_joint: origin xyz=0.0 0.0 0.0 rpy=-1.5707963267948966 0.0 -1.5707963267948966 -> xyz=0 0 0 rpy=-1.5707963267948966 0 -1.5707963267948966
- joint camera_joint: origin xyz=0.15 0.0 0.03 rpy=0.0 0.5 0.0 -> xyz=0.15 0 0.03 rpy=0 0.50 0
- joint camera_left_ir_joint: origin xyz=0.0 0.0 0.0 rpy=0.0 0.0 0.0 -> xyz=0 0.0 0 rpy=0 0 0
- joint camera_left_ir_optical_joint: origin xyz=0.0 0.0 0.0 rpy=-1.5707963267948966 0.0 -1.5707963267948966 -> xyz=0 0 0 rpy=-1.5707963267948966 0 -1.5707963267948966
- joint camera_link_joint: origin xyz=0.0 0.0175 0.0125 rpy=0.0 0.0 0.0 -> xyz=0 0.0175 0.0125 rpy=0 0 0
- joint camera_right_ir_joint: origin xyz=0.0 -0.05 0.0 rpy=0.0 0.0 0.0 -> xyz=0 -0.05 0 rpy=0 0 0
- joint camera_right_ir_optical_joint: origin xyz=0.0 0.0 0.0 rpy=-1.5707963267948966 0.0 -1.5707963267948966 -> xyz=0 0 0 rpy=-1.5707963267948966 0 -1.5707963267948966
- joint floating_base: origin xyz=0.0 0.0 0.0 rpy=0.0 0.0 0.0 -> xyz=0 0 0 rpy=0 0 0
- joint imu_joint: origin xyz=-0.01592 -0.06659 -0.00617 rpy=0.0 0.0 0.0 -> xyz=-0.01592 -0.06659 -0.00617 rpy=0 0 0
- joint optitrack: axis 0.0 0.0 0.0 -> 0 0 0; origin xyz=0.000100572552861879 0.055230109658504 0.1138 rpy=0.0 0.0 0.0 -> xyz=0.000100572552861879 0.055230109658504 0.1138 rpy=0 0 0
- joint rebar_tying_frame: origin xyz=0.2307 -0.0112 -0.190252 rpy=0.0 0.0 0.0 -> xyz=0.2307 -0.0112 -0.190252 rpy=0 0 0
- joint trunk_oriented: origin xyz=0.0 0.0 0.0 rpy=0.0 0.0 1.5707 -> xyz=0 0 0 rpy=0 0 1.5707
